Commit message: added rounded finger t42s

File: t42/pin_flexure_round/t42_flexure.urdf (robot description, URDF)
Before this commit: robot t42, 8 links, 7 joints
Links:
- link distal_l: geometry collision mesh filename=package://openhand_simulation/t42/pin_flexure_round/t42_rou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 scale=0.001 0.001 0.001; visual mesh filename=package://openhand_simulation/t42/pin_flexure_round/t42_rou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 scale=0.001 0.001 0.001
- link distal_r: geometry collision mesh filename=package://openhand_simulation/t42/pin_flexure_round/t42_rou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 scale=0.001 0.001 0.001; visual mesh filename=package://openhand_simulation/t42/pin_flexure_round/t42_rou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 scale=0.001 0.001 0.001
- link hand_coupler: geometry collision cylinder length=0.02562 radius=0.05715; visual cylinder length=0.02562 radius=0.05715
- link prox_l: geometry collision box size=0.038100 0.019050 0.078740; visual mesh filename=package://openhand_simulation/t42/pin_flexure_round/t42_rou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 scale=0.001 0.001 0.001
- link prox_r: geometry collision box size=0.038100 0.019050 0.078740; visual mesh filename=package://openhand_simulation/t42/pin_flexure_round/t42_rou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 scale=0.001 0.001 0.001
Joints:
- joint fixed1: origin xyz=-0.008890 0.000000 0.000000 rpy=0 0 0 -> xyz=-0.01281 0.000000 0.000000 rpy=0 0 0
- joint fixed2: origin xyz=-0.029210 0.000000 0.000000 rpy=0 0 0 -> xyz=-0.03821 0.000000 0.000000 rpy=0 0 0
